Commit message: blog 2 update

File: swarm_follow_leader/urdf/neato.urdf.xacro (robot description, xacro)
@@ -6,10 +6,11 @@
       neato_description/launch/view_model.launch
  -->
-<robot name="neato" xmlns:xacro="http://ros.org/wiki/xacro">
+<robot name="neato"
+  xmlns:xacro="http://ros.org/wiki/xacro">
   <xacro:include filename="$(find swarm_follow_leader)/urdf/common_properties.urdf.xacro"/>
   <xacro:include filename="$(find swarm_follow_leader)/urdf/neato_gazebo.urdf.xacro"/>
   <!-- neato -->
   <xacro:macro name="neato">
-	  <xacro:property name="camera_link" value="0.05" />
+    <xacro:property name="camera_link" value="0.05" />
     <link name="base_footprint"/>
     <joint name="base_joint" type="fixed">
@@ -46,4 +47,19 @@
       </inertial>
     </link>
+    <link name='marker_link'>
+      <visual>
+        <geometry>
+          <mesh filename="model://marker0/meshes/Marker0.dae" scale="0.4 0.4 0.4"/>
+        </geometry>
+        <origin xyz="0 0 0.4" rpy="${M_PI/2} 0 0"/>
+      </visual>
+    </link>
+    <joint name='marker_joint' type='fixed'>
+      <parent link="base_footprint"/>
+      <child link="marker_link"/>
+"
+      <origin xyz="0.00 ${0.235/2} 0.0250" rpy="0 0 0"/>
+      <axis xyz="0 1 0"/>
+    </joint>
     <joint name="wheel_left_joint" type="continuous">
       <parent link="base_link"/>
@@ -95,7 +111,5 @@
         <mass value="0.01" />
         <origin xyz="0 0 0" />
-        <inertia ixx="0.001" ixy="0.0" ixz="0.0"
-                 iyy="0.001" iyz="0.0"
-                 izz="0.001" />
+        <inertia ixx="0.001" ixy="0.0" ixz="0.0" iyy="0.001" iyz="0.0" izz="0.001" />
       </inertial>
     </link>
@@ -115,7 +129,5 @@
         <mass value="0.01" />
         <origin xyz="0 0 0" />
-        <inertia ixx="0.001" ixy="0.0" ixz="0.0"
-                 iyy="0.001" iyz="0.0"
-                 izz="0.001" />
+        <inertia ixx="0.001" ixy="0.0" ixz="0.0" iyy="0.001" iyz="0.0" izz="0.001" />
       </inertial>
     </link>
@@ -135,7 +147,5 @@
         <mass value="0.01" />
         <origin xyz="0 0 0" />
-        <inertia ixx="0.001" ixy="0.0" ixz="0.0"
-                 iyy="0.001" iyz="0.0"
-                 izz="0.001" />
+        <inertia ixx="0.001" ixy="0.0" ixz="0.0" iyy="0.001" iyz="0.0" izz="0.001" />
       </inertial>
     </link>
@@ -155,7 +165,5 @@
         <mass value="0.01" />
         <origin xyz="0 0 0" />
-        <inertia ixx="0.001" ixy="0.0" ixz="0.0"
-                 iyy="0.001" iyz="0.0"
-                 izz="0.001" />
+        <inertia ixx="0.001" ixy="0.0" ixz="0.0" iyy="0.001" iyz="0.0" izz="0.001" />
       </inertial>
     </link>
@@ -175,7 +183,5 @@
         <mass value="0.01" />
         <origin xyz="0 0 0" />
-        <inertia ixx="0.001" ixy="0.0" ixz="0.0"
-                 iyy="0.001" iyz="0.0"
-                 izz="0.001" />
+        <inertia ixx="0.001" ixy="0.0" ixz="0.0" iyy="0.001" iyz="0.0" izz="0.001" />
       </inertial>
     </link>
@@ -191,7 +197,5 @@
         <mass value="0.001"/>
         <origin xyz="0 0 0" rpy="0 0 0"/>
-        <inertia ixx="0.0001" ixy="0" ixz="0"
-                 iyy="0.000001" iyz="0"
-                 izz="0.0001"/>
+        <inertia ixx="0.0001" ixy="0" ixz="0" iyy="0.000001" iyz="0" izz="0.0001"/>
       </inertial>
     </link>
@@ -205,7 +209,5 @@
         <mass value="0.0001" />
         <origin xyz="0 0 0" />
-        <inertia ixx="0.0001" ixy="0.0" ixz="0.0"
-                 iyy="0.0001" iyz="0.0"
-                 izz="0.0001" />
+        <inertia ixx="0.0001" ixy="0.0" ixz="0.0" iyy="0.0001" iyz="0.0" izz="0.0001" />
       </inertial>
     </link>
@@ -219,7 +221,5 @@
         <mass value="0.0001" />
         <origin xyz="0 0 0" />
-        <inertia ixx="0.0001" ixy="0.0" ixz="0.0"
-                 iyy="0.0001" iyz="0.0"
-                 izz="0.0001" />
+        <inertia ixx="0.0001" ixy="0.0" ixz="0.0" iyy="0.0001" iyz="0.0" izz="0.0001" />
       </inertial>
     </link>
@@ -235,37 +235,35 @@
         <mass value="0.0001" />
         <origin xyz="0 0 0"/>
-        <inertia ixx="0.0001" ixy="0.0" ixz="0.0"
-                 iyy="0.0001" iyz="0.0"
-                 izz="0.0001" />
-      </inertial>
-    </link>
-<xacro:if value="$(arg load_camera)">
-  <joint name="camera_joint" type="fixed">
-    <axis xyz="0 1 0" />
-    <origin xyz="-0.1 0 0.25" rpy="0 0 0"/>
-    <parent link="base_link"/>
-    <child link="camera_link"/>
-  </joint>
-  <link name="camera_link">
-    <collision>
-      <origin xyz="0 0 0" rpy="0 0 0"/>
-      <geometry>
-    <box size="${camera_link} ${camera_link} ${camera_link}"/>
-      </geometry>
-    </collision>
-    <visual>
-      <origin xyz="0 0 0" rpy="0 0 0"/>
-      <geometry>
-    <box size="${camera_link} ${camera_link} ${camera_link}"/>
-      </geometry>
-      <material name="red"/>
-    </visual>
-    <inertial>
-      <mass value="1e-5" />
-      <origin xyz="0 0 0" rpy="0 0 0"/>
-      <inertia ixx="1e-6" ixy="0" ixz="0" iyy="1e-6" iyz="0" izz="1e-6" />
-    </inertial>
-  </link>
-</xacro:if>
+        <inertia ixx="0.0001" ixy="0.0" ixz="0.0" iyy="0.0001" iyz="0.0" izz="0.0001" />
+      </inertial>
+    </link>
+    <xacro:if value="$(arg load_camera)">
+      <joint name="camera_joint" type="fixed">
+        <axis xyz="0 1 0" />
+        <origin xyz="-0.1 0 0.25" rpy="0 0 0"/>
+        <parent link="base_link"/>
+        <child link="camera_link"/>
+      </joint>
+      <link name="camera_link">
+        <collision>
+          <origin xyz="0 0 0" rpy="0 0 0"/>
+          <geometry>
+            <box size="${camera_link} ${camera_link} ${camera_link}"/>
+          </geometry>
+        </collision>
+        <visual>
+          <origin xyz="0 0 0" rpy="0 0 0"/>
+          <geometry>
+            <box size="${camera_link} ${camera_link} ${camera_link}"/>
+          </geometry>
+          <material name="red"/>
+        </visual>
+        <inertial>
+          <mass value="1e-5" />
+          <origin xyz="0 0 0" rpy="0 0 0"/>
+          <inertia ixx="1e-6" ixy="0" ixz="0" iyy="1e-6" iyz="0" izz="1e-6" />
+        </inertial>
+      </link>
+    </xacro:if>
     <xacro:neato_sim/>
   </xacro:macro>

Commit message: add lidar target

File: swarm_follow_leader/urdf/neato.urdf.xacro (robot description, xacro)
@@ -62,4 +62,16 @@
       <axis xyz="0 1 0"/>
     </joint>
+      <link name="lidar_target_link">
+    <visual>
+      <geometry>
+        <box size="0.05 0.05 0.2"/>
+      </geometry>
+      <origin xyz="-0.1 0 0.1" rpy="${M_PI/2} 0 0"/>
+    </visual>
+  </link>
+    <joint name="lidar_target_joint" type="fixed">
+    <parent link="base_footprint"/>
+    <child link="lidar_target_link"/>
+  </joint>
     <joint name="wheel_left_joint" type="continuous">
       <parent link="base_link"/>

Commit message: Update follower to use formation engine and use namespace for vision

File: swarm_follow_leader/urdf/neato.urdf.xacro (robot description, xacro)
@@ -50,5 +50,5 @@
       <visual>
         <geometry>
-          <mesh filename="model://marker0/meshes/Marker0.dae" scale="0.4 0.4 0.4"/>
+          <mesh filename="package://swarm_follow_leader/models/marker0/meshes/Marker0.dae" scale="0.4 0.4 0.4"/>
         </geometry>
         <origin xyz="0 0 0.4" rpy="${M_PI/2} 0 0"/>

Commit message: adjust lidar target

File: swarm_follow_leader/urdf/neato.urdf.xacro (robot description, xacro)
@@ -65,7 +65,7 @@
     <visual>
       <geometry>
-        <box size="0.05 0.05 0.2"/>
+        <box size="0.05 0.1 0.2"/>
       </geometry>
-      <origin xyz="-0.1 0 0.1" rpy="${M_PI/2} 0 0"/>
+      <origin xyz="-0.1 0 0.12" rpy="${M_PI/2} 0 0"/>
     </visual>
   </link>

Commit message: border and more robust detection

File: swarm_follow_leader/urdf/neato.urdf.xacro (robot description, xacro)
@@ -47,4 +47,19 @@
       </inertial>
     </link>
+    <link name='border_link'>
+      <visual>
+        <geometry>
+          <box size="0.01 0.25 0.25"/>
+        </geometry>
+        <origin xyz="0.01 -0.1 0.4" rpy="${M_PI/2} 0 0"/>
+      </visual>
+    </link>
+    <joint name='border_joint' type='fixed'>
+      <parent link="base_footprint"/>
+      <child link="border_link"/>
+"
+      <origin xyz="0.00 ${0.235/2} 0.0250" rpy="0 0 0"/>
+      <axis xyz="0 1 0"/>
+    </joint>
     <link name='marker_link'>
       <visual>
